File: TweakTone_V1-2.kicad_pcb (KiCad board)
At the start: 2 copper layers, 65.9 x 60.6 mm, 57 parts, among them IC1 PT2399, IC2 TL072, M1 PAD8, M2 PAD8

Commit message: update
Parts:
- +9V0, GND0: footprint SQUARE -> TweakTone_V1-2:SQUARE
- moved +9V0 11.9 mm to (174.2, 92.5)
- moved L+0 11.4 mm to (159.0, 90.9)
- moved R1 8.59 mm to (137.5, 135.3), turned to 90 degrees
- moved R2 4.07 mm to (145.7, 136.7), turned to -90 degrees
- moved R19 3.94 mm to (145.4, 144.4)
- moved R3 3.49 mm to (149.0, 134.7), turned to 90 degrees
- moved C1 3.43 mm to (143.1, 129.8)
- moved IN0 3.22 mm to (140.7, 126.5)
- moved R16 1.27 mm to (196.6, 107.7)
- moved C11 1.27 mm to (192.5, 114.8)
- moved C12 0.92 mm to (191.4, 96.0)
- moved C21 0.46 mm to (175.3, 98.0)
- moved R18 0.17 mm to (166.6, 92.5), turned to 0 degrees
Connections:
- +9V0 pad 1: +9V -> +9V(T)
Routing:
- net +9V: track 71.7 -> 0.00 mm
- net +9V(T): track 0.00 -> 65.7 mm
- net (no net): track 16.2 -> 0.00 mm
- net Net-(IN0-PAD): track 17.9 -> 7.09 mm
- net Net-(C11-Pad2): track 0.00 -> 9.91 mm
- net Net-(IC2A--IN): track 6.26 -> 12.9 mm
- net GND: track 15.9 -> 11.3 mm
- net Net-(C12-Pad1): track 18.3 -> 21.7 mm
- net Net-(IC2A-OUT): track 12.7 -> 16.1 mm
- net Net-(C9-Pad1): track 22.1 -> 19.1 mm
- net VR: track 22.7 -> 25.4 mm
- net Net-(L+0-PAD): track 3.44 -> 4.44 mm
- added copper zone on B.Cu, net GND
Other:
- outline, holes or cut-outs redrawn

Commit message: fix missing connection between MIX0 and wet signal
Connections:
- MIX0 pad 3: unconnected-(MIX0-Pad3) -> Net-(C11-Pad2)
Routing:
- net Net-(C11-Pad2): track 9.91 -> 15.9 mm
